File: GRUB.kicad_sch (KiCad schematic)
At the start: 54 parts, among them J1 External controller, timer or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, J2 A/C, J3 LEDs Drivers Connector, Q1 2N3904, Q2 2N3904, Q3 2N3904, Q5 2N3904, SW1 R_SWITCH, SW2 U_SWITCH, SW3 B_SWITCH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

Commit message: Adding power rack schematic
Parts:
- removed J2: A/C, symbol Connector:Screw_Terminal_01x03
- removed PS1: HS-40024, Converter_ACDC:Converter_ACDC_Hahn_HS-400xx_THT, symbol Converter_ACDC:HS-40024
- R10, R12, R13, R7: value R -> 220
- R11, R14, R15, R16, R2, R3, R4, R5: value 2k -> 220
Other:
- sheet LEDs drivers renamed LEDs_drivers
- added sheet Power (Power.kicad_sch)
- note removed: "24V"
- note removed: "at least 40W"
